File: BeeWeight_MKRWAN/BeeWeight_MKRWAN.sch (KiCad schematic (older format))
At the start: 34 parts, among them J2 691412120004B, J3 691412120004B, J4 691412120004B, J5 691412120004B, J6 Conn_01x02_Male, J7 Conn_01x14_Female, J8 Conn_01x14_Female, J9 694108301002, Q1 IRLML2244, U1 ADS1241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

Commit message: Update Crystal Footprint
Parts:
- Y1: footprint USMB_Syl_Mont:Crystal_4Mhz_MCRSD04000F183000RR -> USMB_Syl_Mont:Crystal-4Mhz-TH-Wurth-830027298B
Changed lines of the file:
@@
 F 0 "Y1" H 10300 2668 50  0000 C CNN
 F 1 "Crystal" H 10300 2577 50  0000 C CNN
-F 2 "USMB_Syl_Mont:Crystal_4Mhz_MCRSD04000F183000RR" H 10300 2400 50  0001 C CNN
+F 2 "USMB_Syl_Mont:Crystal-4Mhz-TH-Wurth-830027298B" H 10300 2400 50  0001 C CNN
 F 3 "~" H 10300 2400 50  0001 C CNN
 	1    10300 2400

Commit message: Minor changes in schematic and PCB
Parts:
- Q1: value IRLML2244 -> IRLML6244
Connections:
- wire segments 140 -> 139
Changed lines of the file:
@@
 P 5725 3750
 F 0 "Q1" H 5929 3796 50  0000 L CNN
-F 1 "IRLML2244" H 5929 3705 50  0000 L CNN
+F 1 "IRLML6244" H 5929 3705 50  0000 L CNN
 F 2 "Package_TO_SOT_SMD:SOT-23" H 5925 3675 50  0001 L CIN
-F 3 "https://www.infineon.com/dgdl/irlml2060pbf.pdf?fileId=5546d462533600a401535664b7fb25ee" H 5725 3750 50  0001 L CNN
+F 3 "https://fr.rs-online.com/web/p/transistors-mosfet/7377228/" H 5725 3750 50  0001 L CNN
 	1    5725 3750
 	1    0    0    -1
@@
 Wire Wire Line
 	7900 6125 6025 6125
-Connection ~ 5675 6125
-Wire Wire Line
-	5675 6125 5650 6125
 Wire Wire Line
 	6025 6100 6025 6125
-Connection ~ 6025 6125
-Wire Wire Line
-	6025 6125 5675 6125
 Wire Notes Line
 	4325 4975 6675 4975
@@
 Wire Wire Line
 	5650 3425 5525 3425
+Wire Wire Line
+	5675 6125 6025 6125
+Connection ~ 6025 6125
 $EndSCHEMATC

Commit message: Nouveau routage par G.Manusset
Parts:
- added JP1: SolderJumper_2_Open, Jumper:SolderJumper-2_P1.3mm_Open_RoundedPad1.0x1.5mm, symbol Jumper:SolderJumper_2_Open
- J2, J3, J4, J5: symbol TermBlock_1x04_P3.50mm_Wurth_691412120004B:691412120004B -> BeeWeight_MKRWAN-rescue:691412120004B-TermBlock_1x04_P3.50mm_Wurth_691412120004B
- J9: symbol Jack_DC_2.1mm_Wurth_694108301002:694108301002 -> BeeWeight_MKRWAN-rescue:694108301002-Jack_DC_2.1mm_Wurth_694108301002
- U1: symbol USMB_Syl_Mont:ADS1241 -> BeeWeight_MKRWAN-rescue:ADS1241-USMB_Syl_Mont
Connections:
- net GND: now also JP1.2 (B)
- net GND_LowPower: now also JP1.1 (A)
Other:
- moved on the sheet: Q1, R1
Changed lines of the file:
@@
 $EndDescr
 $Comp
-L USMB_Syl_Mont:ADS1241 U1
+L BeeWeight_MKRWAN-rescue:ADS1241-USMB_Syl_Mont U1
 U 1 1 6081276C
 P 8525 3125
@@
 AREF
 $Comp
-L Transistor_FET:IRLML2060 Q1
-U 1 1 608900FB
-P 5725 3750
-F 0 "Q1" H 5929 3796 50  0000 L CNN
-F 1 "IRLML6244" H 5929 3705 50  0000 L CNN
-F 2 "Package_TO_SOT_SMD:SOT-23" H 5925 3675 50  0001 L CIN
-F 3 "https://fr.rs-online.com/web/p/transistors-mosfet/7377228/" H 5725 3750 50  0001 L CNN
-	1    5725 3750
-	1    0    0    -1
-$EndComp
-Wire Wire Line
-	5825 3950 5825 4175
-$Comp
 L power:GND #PWR02
 U 1 1 608A656C
-P 5825 4175
-F 0 "#PWR02" H 5825 3925 50  0001 C CNN
-F 1 "GND" H 5830 4002 50  0000 C CNN
-F 2 "" H 5825 4175 50  0001 C CNN
-F 3 "" H 5825 4175 50  0001 C CNN
-	1    5825 4175
-	1    0    0    -1
-$EndComp
-Text Label 5525 3425 2    50   ~ 0
-GND_LowPower
+P 5750 4200
+F 0 "#PWR02" H 5750 3950 50  0001 C CNN
+F 1 "GND" H 5755 4027 50  0000 C CNN
+F 2 "" H 5750 4200 50  0001 C CNN
+F 3 "" H 5750 4200 50  0001 C CNN
+	1    5750 4200
+	1    0    0    -1
+$EndComp
 $Comp
 L power:GND #PWR03
@@
 Wire Wire Line
 	7800 6025 7900 6025
-Text Label 5100 3750 2    50   ~ 0
-D3_CMD_MOS
 Text Label 5375 6525 0    50   ~ 0
 GND_LowPower
@@
 	1    0    0    -1
 $EndComp
-Wire Wire Line
-	5825 3425 5825 3550
-Wire Wire Line
-	5825 3425 5650 3425
-$Comp
-L Device:R R1
-U 1 1 608E9B92
-P 5325 3975
-F 0 "R1" H 5395 4021 50  0000 L CNN
-F 1 "1M" H 5395 3930 50  0000 L CNN
-F 2 "Resistor_SMD:R_0805_2012Metric_Pad1.15x1.40mm_HandSolder" V 5255 3975 50  0001 C CNN
-F 3 "~" H 5325 3975 50  0001 C CNN
-	1    5325 3975
-	-1   0    0    1
-$EndComp
-Wire Wire Line
-	5325 3750 5525 3750
-Wire Wire Line
-	5325 4175 5825 4175
-Connection ~ 5825 4175
-Wire Wire Line
-	5325 3825 5325 3750
-Wire Wire Line
-	5325 4125 5325 4175
-Wire Wire Line
-	5325 3750 5100 3750
-Connection ~ 5325 3750
 $Comp
 L Device:C C9
@@
 	2225 3500 2075 3500
 $Comp
-L TermBlock_1x04_P3.50mm_Wurth_691412120004B:691412120004B J5
+L BeeWeight_MKRWAN-rescue:691412120004B-TermBlock_1x04_P3.50mm_Wurth_691412120004B J5
 U 1 1 608E7BAB
 P 2425 3400
@@
 	2200 4650 2050 4650
 $Comp
-L TermBlock_1x04_P3.50mm_Wurth_691412120004B:691412120004B J4
+L BeeWeight_MKRWAN-rescue:691412120004B-TermBlock_1x04_P3.50mm_Wurth_691412120004B J4
 U 1 1 60985811
 P 2400 4550
@@
 	2150 5825 2000 5825
 $Comp
-L TermBlock_1x04_P3.50mm_Wurth_691412120004B:691412120004B J2
+L BeeWeight_MKRWAN-rescue:691412120004B-TermBlock_1x04_P3.50mm_Wurth_691412120004B J2
 U 1 1 60999B34
 P 2350 5725
@@
 	2150 7000 2000 7000
 $Comp
-L TermBlock_1x04_P3.50mm_Wurth_691412120004B:691412120004B J3
+L BeeWeight_MKRWAN-rescue:691412120004B-TermBlock_1x04_P3.50mm_Wurth_691412120004B J3
 U 1 1 609ACB49
 P 2350 6900
@@
 NoConn ~ 9225 5325
 $Comp
-L Jack_DC_2.1mm_Wurth_694108301002:694108301002 J9
+L BeeWeight_MKRWAN-rescue:694108301002-Jack_DC_2.1mm_Wurth_694108301002 J9
 U 1 1 60ABF432
 P 1625 1500
@@
 L power:PWR_FLAG #FLG0103
 U 1 1 60CE6733
-P 5650 3375
-F 0 "#FLG0103" H 5650 3450 50  0001 C CNN
-F 1 "PWR_FLAG" H 5650 3548 50  0000 C CNN
-F 2 "" H 5650 3375 50  0001 C CNN
-F 3 "~" H 5650 3375 50  0001 C CNN
-	1    5650 3375
-	1    0    0    -1
-$EndComp
-Wire Wire Line
-	5650 3375 5650 3425
-Connection ~ 5650 3425
-Wire Wire Line
-	5650 3425 5525 3425
+P 5600 3400
+F 0 "#FLG0103" H 5600 3475 50  0001 C CNN
+F 1 "PWR_FLAG" H 5600 3573 50  0000 C CNN
+F 2 "" H 5600 3400 50  0001 C CNN
+F 3 "~" H 5600 3400 50  0001 C CNN
+	1    5600 3400
+	1    0    0    -1
+$EndComp
 Wire Wire Line
 	5675 6125 6025 6125
 Connection ~ 6025 6125
+$Comp
+L Jumper:SolderJumper_2_Open JP1
+U 1 1 609AB68F
+P 6050 3750
+F 0 "JP1" V 6004 3818 50  0000 L CNN
+F 1 "SolderJumper_2_Open" V 6095 3818 50  0000 L CNN
+F 2 "Jumper:SolderJumper-2_P1.3mm_Open_RoundedPad1.0x1.5mm" H 6050 3750 50  0001 C CNN
+F 3 "~" H 6050 3750 50  0001 C CNN
+	1    6050 3750
+	0    1    1    0
+$EndComp
+$Comp
+L Device:R R1
+U 1 1 608E9B92
+P 5300 3950
+F 0 "R1" H 5370 3996 50  0000 L CNN
+F 1 "1M" H 5370 3905 50  0000 L CNN
+F 2 "Resistor_SMD:R_0805_2012Metric_Pad1.15x1.40mm_HandSolder" V 5230 3950 50  0001 C CNN
+F 3 "~" H 5300 3950 50  0001 C CNN
+	1    5300 3950
+	-1   0    0    1
+$EndComp
+Text Label 5100 3750 2    50   ~ 0
+D3_CMD_MOS
+$Comp
+L Transistor_FET:IRLML2060 Q1
+U 1 1 608900FB
+P 5650 3750
+F 0 "Q1" H 5475 3650 50  0000 L CNN
+F 1 "IRLML6244" H 5475 3550 50  0000 L CNN
+F 2 "Package_TO_SOT_SMD:SOT-23" H 5850 3675 50  0001 L CIN
+F 3 "https://fr.rs-online.com/web/p/transistors-mosfet/7377228/" H 5650 3750 50  0001 L CNN
+	1    5650 3750
+	1    0    0    -1
+$EndComp
+Wire Wire Line
+	5750 3550 5750 3500
+Wire Wire Line
+	5750 3400 5600 3400
+Connection ~ 5600 3400
+Wire Wire Line
+	5600 3400 5250 3400
+Text Label 5250 3400 2    50   ~ 0
+GND_LowPower
+Wire Wire Line
+	5750 4200 5750 4150
+Wire Wire Line
+	5450 3750 5300 3750
+Wire Wire Line
+	5300 3800 5300 3750
+Connection ~ 5300 3750
+Wire Wire Line
+	5300 3750 5100 3750
+Wire Wire Line
+	5300 4100 5300 4150
+Wire Wire Line
+	5300 4150 5750 4150
+Connection ~ 5750 4150
+Wire Wire Line
+	5750 4150 5750 4000
+Wire Wire Line
+	6050 3600 6050 3500
+Wire Wire Line
+	6050 3500 5750 3500
+Connection ~ 5750 3500
+Wire Wire Line
+	5750 3500 5750 3400
+Wire Wire Line
+	5750 4000 6050 4000
+Wire Wire Line
+	6050 4000 6050 3900
+Connection ~ 5750 4000
+Wire Wire Line
+	5750 4000 5750 3950
 $EndSCHEMATC

Commit message: Update DS18B20 Footprint
Otherwise eurocircuit fees are based on class 8 PCB
Parts:
- U2: footprint Package_TO_SOT_THT:TO-92_Inline -> Package_TO_SOT_THT:TO-92
Changed lines of the file:
@@
 F 0 "U2" H 5145 6171 50  0000 R CNN
 F 1 "DS18B20" H 5145 6080 50  0000 R CNN
-F 2 "Package_TO_SOT_THT:TO-92_Inline" H 4375 5875 50  0001 C CNN
+F 2 "Package_TO_SOT_THT:TO-92" H 4375 5875 50  0001 C CNN
 F 3 "http://datasheets.maximintegrated.com/en/ds/DS18B20.pdf" H 5225 6375 50  0001 C CNN
 	1    5375 6125
